File: MRR_ESPA/current/MRR_ESPA.kicad_pcb (KiCad board)
At the start: 2 copper layers, 99.5 x 99.5 mm, 135 parts, among them J1 X_MIN, J10 PART_FAN, J11 FAN_HEATSINK, J12 T_BED, J13 T_E0, J14 I2C/SPI, J15 AUX1, J16 USB_B_Micro, J17 Serial, J18 PINS_1, J19 PINS_2, J2 Z_MIN, J20 CS_PINS, J21 X_MOTOR, J22 Z_MOTOR, J23 Y_MOTOR, J24 E0_MOTOR, J3 BED, J4 Micro_SD_Card_China, J5 Y_MIN, J6 Z_PROBE, J7 E0, J8 FAN_CASE, J9 PWR_IN, Q1 IRLS3034PBF, Q2 IRLR8743TRPBF, Q3 IRLR8743TRPBF, Q4 S9014, Q5 S9014, SW1 RESET, U1 ESP32-WROOM-32D, U10 TLP182, U11 74LVC1G125, U12 74LVC1G125, U2 TPS54340DDA, U3 CH340C, U4 AMS1117-3.3, U5 Pololu_board, U6 Pololu_board, U7 TXS0102DCUR, U8 Pololu_board, U9 Pololu_board

Commit message: Added v1.0
Parts:
- removed C20, C21: 100nF16V, Capacitor_SMD:C_0805_2012Metric
- removed J20: CS_PINS, Connector_PinHeader_2.54mm:PinHeader_1x04_P2.54mm_Vertical
- removed U7: TXS0102DCUR, Package_SO:VSSOP-8_2.4x2.1mm_P0.5mm
- added R7: 2.2K, Resistor_SMD:R_0805_2012Metric, F.Cu at (97.7, 81.8)
- R6: value 1K -> 1.5K
- moved F2 18.5 mm to (124.5, 88.8), turned to 90 degrees
- moved D10 18.0 mm to (121.8, 61.0), turned to 180 degrees
- moved C14 14.5 mm to (119.1, 48.8)
- moved U4 14.3 mm to (119.1, 54.6)
- moved R28 14.1 mm to (118.3, 61.0), turned to 180 degrees
- moved D4 12.3 mm to (123.9, 77.7), turned to 90 degrees
- moved D15 10.7 mm to (127.7, 56.6), turned to 90 degrees
- moved R31 6.85 mm to (121.5, 80.7), turned to 270 degrees
- moved R6 6.42 mm to (97.7, 79.9), turned to 180 degrees
- moved D1 5.71 mm to (127.8, 95.1), turned to 90 degrees
- moved D14 5.48 mm to (125.1, 56.6), turned to 90 degrees
- moved R5 5.28 mm to (127.8, 91.6)
- moved D13 5.06 mm to (121.5, 77.0), turned to 270 degrees
- moved R30 4.61 mm to (130.8, 59.5), turned to 180 degrees
- moved R38 3.05 mm to (104.0, 86.2)
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Connections:
- J15 pad 6: UARTD5V+ -> UARTD+
- J15 pad 8: UARTD5V- -> Net-(J15-Pad8)
- J16 pad 6: (no net) -> GND
- J9 pad 3: Net-(F2-Pad2) -> GNDD
- J9 pad 4: GNDD -> Net-(F2-Pad2)
- JP1 pad 1: MOSI -> +3V3
- JP1 pad 3: +3V3 -> GND
- JP10 pad 1: Y_CS -> +3V3
- JP10 pad 3: +3V3 -> GND
- JP11 pad 1: Z_CS -> +3V3
- JP11 pad 3: +3V3 -> GND
- JP12 pad 1: E0_CS -> +3V3
- JP12 pad 3: +3V3 -> GND
- JP13 pad 1: MISO -> GND
- JP14 pad 1: MISO -> GND
- JP15 pad 1: MISO -> GND
- JP16 pad 1: MISO -> GND
- JP2 pad 1: MOSI -> +3V3
- JP2 pad 3: +3V3 -> GND
- JP3 pad 1: MOSI -> +3V3
- JP3 pad 3: +3V3 -> GND
- JP4 pad 1: MOSI -> +3V3
- JP4 pad 3: +3V3 -> GND
- JP5 pad 1: SCK -> +3V3
- JP5 pad 3: +3V3 -> GND
- JP6 pad 1: SCK -> +3V3
- JP6 pad 3: +3V3 -> GND
- JP7 pad 1: SCK -> +3V3
- JP7 pad 3: +3V3 -> GND
- JP8 pad 1: SCK -> +3V3
- JP8 pad 3: +3V3 -> GND
- JP9 pad 1: X_CS -> +3V3
- JP9 pad 3: +3V3 -> GND
- R6 pad 1: +3V3 -> Net-(J15-Pad8)
- R6 pad 2: GND -> UARTD-
Routing:
- net MISO: track 220.3 -> 54.5 mm, vias 9 -> 1
- net MOSI: track 215.3 -> 58.9 mm, vias 6 -> 2
- net SCK: track 195.0 -> 51.5 mm, vias 7 -> 1
- net GND: track 117.9 -> 189.5 mm, vias 46 -> 84
- net GNDD: track 67.0 -> 9.87 mm, vias 3 -> 0
- net E0_CS: track 44.4 -> 0.00 mm
- net VIN: track 318.6 -> 358.1 mm, vias 10 -> 31
- net +3V3: track 445.0 -> 482.8 mm, vias 15 -> 16
- net VBED: track 75.5 -> 41.5 mm, vias 3 -> 0
- net X_CS: track 28.5 -> 0.00 mm
- net Net-(D1-Pad1): track 28.9 -> 0.88 mm, vias 59 -> 40
- net Z_CS: track 25.1 -> 0.00 mm
- net UARTD5V+: track 20.2 -> 0.00 mm, vias 2 -> 0
- net UARTD5V-: track 18.7 -> 0.00 mm
- net Net-(J15-Pad8): track 0.00 -> 17.7 mm
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- added copper zone on F.Cu, net Net-(D6-Pad1)
- added copper zone on B.Cu, net Net-(F1-Pad2)
- added copper zone on F.Cu, net Net-(F1-Pad2)
Other:
- net class 5V: trace_width 0.3 -> 0.8
- net class VBED: trace_width 2 -> 3; via_dia 0.8 -> 3; via_drill 0.4 -> 2
- board text added: "Developed by Maple Rain Research Co., Ltd."
- board text added: "HEAT BED"
- board text added: "HOT END"
- board text added: "MRR ESPA v1.0"
- board text added: "SLP"
- board text added: "VIO"
- board text added: "Version date: 2019-03-17"
- board text removed: "MRR ESPA v0.9"
- board text removed: "SPI"
- board text removed: "TMC"
- board text removed: "X"
- board text removed: "Y"
- board text removed: "Z"

Commit message: Added macrocfg.json
Parts:
- moved R5 8.42 mm to (121.4, 86.1)
- moved D1 8.37 mm to (121.4, 89.7)
- moved J3 5.33 mm to (132.5, 88.8)
- moved J7 5.33 mm to (132.5, 99.6)
- moved J9 5.33 mm to (132.5, 68.0)
- moved Q2 4.32 mm to (117.5, 100.0)
- moved R9 4.18 mm to (126.0, 99.0), turned to 90 degrees
- moved D3 3.60 mm to (126.0, 102.5), turned to 90 degrees
- moved R10 3.56 mm to (108.4, 96.6)
- moved R11 3.56 mm to (108.5, 98.7)
- moved Q3 2.29 mm to (117.5, 107.6)
- moved R13 2.29 mm to (109.5, 105.2)
- moved R14 2.29 mm to (109.5, 107.3)
Routing:
- net VIN: track 358.1 -> 370.0 mm
- net Net-(D1-Pad1): track 0.88 -> 4.21 mm, vias 40 -> 62
- net VBED: track 41.5 -> 44.3 mm, vias 0 -> 15
- net Net-(D3-Pad1): track 14.0 -> 11.4 mm
- net Net-(D6-Pad1): track 37.3 -> 35.7 mm
- net GND: track 189.5 -> 188.5 mm, vias 84 -> 82
- net +5V: track 140.2 -> 139.3 mm
- net TO_HEATER_E0: track 4.01 -> 4.88 mm
- net Net-(F2-Pad2): vias 0 -> 16
- net Net-(F1-Pad2): vias 0 -> 14
- net GNDD: vias 0 -> 20
Other:
- board text added: "MRR ESPA v1.01"
- board text added: "Version date: 2019-06-05"
- board text removed: "MRR ESPA v1.0"
- board text removed: "Version date: 2019-03-17"
