File: MRR_ESPA/current/MRR_ESPA.sch (KiCad schematic (older format))
At the start: 135 parts, among them J1 X_MIN, J10 PART_FAN, J11 FAN_HEATSINK, J12 T_BED, J13 T_E0, J14 I2C/SPI, J15 AUX1, J16 USB_B_Micro, J17 Serial, J18 PINS_1, J19 PINS_2, J2 Z_MIN, J20 CS_PINS, J21 X_MOTOR, J22 Z_MOTOR, J23 Y_MOTOR, J24 E0_MOTOR, J3 BED, J4 Micro_SD_Card_China, J5 Y_MIN, J6 Z_PROBE, J7 E0, J8 FAN_CASE, J9 PWR_IN, Q1 IRLS3034PBF, Q2 IRLR8743TRPBF, Q3 IRLR8743TRPBF, Q4 S9014, Q5 S9014, SW1 RESET, U1 ESP32-WROOM-32D, U10 TLP182, U11 74LVC1G125, U12 74LVC1G125, U2 TPS54340DDA, U3 CH340C, U4 AMS1117-3.3, U5 Pololu_board, U6 Pololu_board, U7 TXS0102DCUR, U8 Pololu_board, U9 Pololu_board

Commit message: Added v1.0
Parts:
- removed C20, C21: 100nF16V, Capacitor_SMD:C_0805_2012Metric, symbol Device:C
- removed J20: CS_PINS, Connector_PinHeader_2.54mm:PinHeader_1x04_P2.54mm_Vertical, symbol Connector_Generic:Conn_01x04
- removed U7: TXS0102DCUR, Package_SO:VSSOP-8_2.4x2.1mm_P0.5mm, symbol projsym:TXS0102DCUR
- added R7: 2.2K, Resistor_SMD:R_0805_2012Metric, symbol Device:R
- R6: value 1K -> 1.5K
Connections:
- net E0_CS is gone; now on net +3V3: JP12.1 (A)
- net UARTD5V+ is gone; now on net UARTD+: J15.6 (Pin_6)
- net X_CS is gone; now on net +3V3: JP9.1 (A)
- net Y_CS is gone; now on net +3V3: JP10.1 (A)
- net Z_CS is gone; now on net +3V3: JP11.1 (A)
- net +3V3: now also JP1.1 (A), JP2.1 (A), JP3.1 (A), JP4.1 (A), JP5.1 (A), JP6.1 (A), JP7.1 (A), JP8.1 (A); no longer JP1.3 (B), JP10.3 (B), JP11.3 (B), JP12.3 (B), JP2.3 (B), JP3.3 (B), JP4.3 (B), JP5.3 (B), JP6.3 (B), JP7.3 (B), JP8.3 (B), JP9.3 (B), R6.1
- net GND: now also J16.6 (Shield), JP1.3 (B), JP10.3 (B), JP11.3 (B), JP12.3 (B), JP13.1 (A), JP14.1 (A), JP15.1 (A), JP16.1 (A), JP2.3 (B), JP3.3 (B), JP4.3 (B), JP5.3 (B), JP6.3 (B), JP7.3 (B), JP8.3 (B), JP9.3 (B), R7.2; no longer R6.2
- net GNDD: now also J9.3 (Pin_3); no longer J9.4 (Pin_4)
- net MISO: no longer JP13.1 (A), JP14.1 (A), JP15.1 (A), JP16.1 (A)
- net MOSI: no longer JP1.1 (A), JP2.1 (A), JP3.1 (A), JP4.1 (A)
- net SCK: no longer JP5.1 (A), JP6.1 (A), JP7.1 (A), JP8.1 (A)
- net UARTD-: now also R6.2, R7.1
- net at F2.2: now also J9.4 (Pin_4); no longer J9.3 (Pin_3)
- net UARTD5V-: no longer names the net of J15.8 (Pin_8)
- net UARTD5V-: now also R6.1
- no-connect marks 21 -> 20
Other:
- note removed: "Bidirectional 3.3V <-> 5V UART"
- note removed: "CS Pins for SPI mode"
- moved on the sheet: D4, F2, J15, R6
